Commit message: add scripts

File: urdf/bot_description.xacro (robot description, xacro)
@@ -34,5 +34,5 @@
 <link name="front_left_wheel_link">
   <xacro:solid_cylinder_inertial
-  rpy="0 0 0" xyz="0 0 0" mass="0.1" radius="${wheel_radius}" length="0.08"
+  rpy="0 0 0" xyz="0 0 0" mass="1" radius="${wheel_radius}" length="0.08"
   />
   <visual>

File: urdf/gazebo_plagin.xacro (robot description, xacro)
@@ -94,13 +94,3 @@
     </sensor>
   </gazebo>
-  <xacro:macro name="set_wheel_friction" params="link friction">
-    <gazebo reference="${link}">
-      <mu1 value="${friction}"/>
-      <mu2 value="${friction}"/>
-      <kp value="100000.0"/>
-      <kd value="10.0"/>
-      <material>Gazebo/Red</material>
-    </gazebo>
-  </xacro:macro>
-  <xacro:set_wheel_friction link="back_wheel_link" friction="0.01"/>
 </robot>
